File: FMU_V.2/FMU_V.2.sch (EAGLE design)
At the start: 322 parts, among them J201 HEADER_1X4, J202 HEADER_1X4, J203 HEADER_1X4, J204 HEADER_1X4, J301 HEADER_1X4, J302 HEADER_1X4, J303 HEADER_1X4, J401 HEADER_1X4, J402 HEADER_1X4, J403 HEADER_1X4, J404 HEADER_1X4, J701 HEADER_1X4, J901 HEADER_1X4, J902 HEADER_1X4, M3_MOUNT1 MOUNT-HOLE3.1MM, M3_MOUNT2 MOUNT-HOLE3.1MM, M3_MOUNT3 MOUNT-HOLE3.1MM, M3_MOUNT4 MOUNT-HOLE3.1MM, U101 STM32F4X7VX, U102 FM25V01, U201 TXS0108TSSOP-20, U202 LT3469, U301 2908-05WB-MG, U302 NUF2042XV6, U303 ADUM5402, U304 MAX13487E, U305 MAX232ECWE, U401 ADUM5402, U402 MAX3051, U403 MAX3051, U502 ICM20608-G, U503 MPU-9250, U504 MPU-6000, U506 MS5611-01BA, U601 BQ24315, U602 BQ24315, U603 LD1117ASTR, U604 LD1117ASTR, U701 STM32F10XCXT6, U801 TXS0108TSSOP-20, U803 LD1117ASTR, U901 LM5005, U902 LM5005, X101 NX3225SA-24.000MHZ-STD-CSR-1, X701 NX3225SA-24.000MHZ-STD-CSR-1

Commit message: Исправленно #2, #3, #5, #8, #9
Parts:
- removed !VBUS_V, !VDD_BRICK, !VDD_SERVO: PAD.04, pixhawk2:PAD.04
- added R103: 10K, pixhawk2:RESISTOR0603-RES
- added R104: 1M, pixhawk2:RESISTOR0603-RES
- added SJ4: (no value), jumper:SJ2W
- R706: value 10K -> 220R
Connections:
- net PB2-BOOT1 renamed PC5
- removed net PRESSURE_SENS: U101PORTC_L.PC5
- removed net VDD_3V3_SENSORS_EN: U101PORTE_L.PE3
- new net N$14: R104.1, U101PORTE_L.PE3
- new net N$16: R103.1, U101PORTC_L.PC5
- net !VBUS_VALID: no longer !VBUS_V.P$1
- net !VDD_BRICK_VALID: now also SJ4.1; no longer !VDD_BRICK.P$1
- net !VDD_SERVO_VALID: now also SJ4.3; no longer !VDD_SERVO.P$1
- net GND: now also R103.2, R104.2, SJ4.2
Other:
- note added: "Buzzer"
- note removed: "+ SIGNAL _"
- moved on the sheet: F-BOOT, IO-BOOT0
Changed lines of the file:
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@@
 <part name="GND77" library="pixhawk2" deviceset="GND" device=""/>
 <part name="GND78" library="pixhawk2" deviceset="GND" device=""/>
-<part name="!VBUS_V" library="pixhawk2" deviceset="PAD" device=".04">
-<attribute name="BOM" value="EXCLUDE"/>
-<attribute name="PARTNO" value="*"/>
-</part>
 <part name="GND81" library="pixhawk2" deviceset="GND" device=""/>
 <part name="GND85" library="pixhawk2" deviceset="GND" device=""/>
@@
 <part name="GND110" library="pixhawk2" deviceset="GND" device=""/>
 <part name="GND9" library="pixhawk2" deviceset="GND" device=""/>
-<part name="!VDD_SERVO" library="pixhawk2" deviceset="PAD" device=".04">
-<attribute name="BOM" value="EXCLUDE"/>
-<attribute name="PARTNO" value="*"/>
-</part>
-<part name="!VDD_BRICK" library="pixhawk2" deviceset="PAD" device=".04">
-<attribute name="BOM" value="EXCLUDE"/>
-<attribute name="PARTNO" value="*"/>
-</part>
 <part name="VDD_5V_IN" library="pixhawk2" deviceset="PAD" device=".04">
 <attribute name="BOM" value="EXCLUDE"/>
@@
 <part name="GND84" library="pixhawk2" deviceset="GND" device=""/>
 <part name="D302" library="fmu2" deviceset="DIODE-SCHOTTKY" device="_MSMP" value="MSS1P4-M3/89A"/>
-<part name="R706" library="pixhawk2" deviceset="RESISTOR" device="0603-RES" value="10K"/>
+<part name="R706" library="pixhawk2" deviceset="RESISTOR" device="0603-RES" value="220R"/>
 <part name="GND58" library="pixhawk2" deviceset="GND" device=""/>
 <part name="C804" library="pixhawk2" deviceset="CAP" device="0603" value="0u1"/>
@@
 <part name="GND45" library="pixhawk2" deviceset="GND" device=""/>
 <part name="USB1" library="pixhawk2" deviceset="MOLEX-47346-0001" device=""/>
+<part name="GND51" library="pixhawk2" deviceset="GND" device=""/>
+<part name="R104" library="pixhawk2" deviceset="RESISTOR" device="0603-RES" value="1M"/>
+<part name="R103" library="pixhawk2" deviceset="RESISTOR" device="0603-RES" value="10K"/>
+<part name="GND53" library="pixhawk2" deviceset="GND" device=""/>
+<part name="SJ4" library="jumper" deviceset="SJ2W" device=""/>
+<part name="GND56" library="pixhawk2" deviceset="GND" device=""/>
 </parts>
 <sheets>
@@
 <instance part="F-DIO" gate="G$1" x="25.4" y="30.48" rot="MR0"/>
 <instance part="F-VDD_3V3" gate="G$1" x="25.4" y="22.86" rot="MR0"/>
+<instance part="GND51" gate="1" x="226.06" y="152.4"/>
+<instance part="R104" gate="G$1" x="215.9" y="157.48"/>
+<instance part="R103" gate="G$1" x="142.24" y="152.4"/>
+<instance part="GND53" gate="1" x="149.86" y="147.32"/>
+<instance part="SJ4" gate="G$1" x="63.5" y="86.36" rot="MR90"/>
+<instance part="GND56" gate="1" x="63.5" y="76.2"/>
 </instances>
 <busses>
@@
 </segment>
 </net>
-<net name="PB2-BOOT1" class="0">
+<net name="PC5" class="0">
 <segment>
 <wire x1="33.02" y1="104.14" x2="63.5" y2="104.14" width="0.1524" layer="91"/>
@@
 <pinref part="C101" gate="G$1" pin="2"/>
 </segment>
+<segment>
+<pinref part="GND51" gate="1" pin="GND"/>
+<wire x1="226.06" y1="154.94" x2="226.06" y2="157.48" width="0.1524" layer="91"/>
+<pinref part="R104" gate="G$1" pin="2"/>
+<wire x1="226.06" y1="157.48" x2="220.98" y2="157.48" width="0.1524" layer="91"/>
+</segment>
+<segment>
+<pinref part="R103" gate="G$1" pin="2"/>
+<wire x1="147.32" y1="152.4" x2="149.86" y2="152.4" width="0.1524" layer="91"/>
+<wire x1="149.86" y1="152.4" x2="149.86" y2="149.86" width="0.1524" layer="91"/>
+<pinref part="GND53" gate="1" pin="GND"/>
+</segment>
+<segment>
+<pinref part="SJ4" gate="G$1" pin="2"/>
+<wire x1="63.5" y1="81.28" x2="63.5" y2="78.74" width="0.1524" layer="91"/>
+<pinref part="GND56" gate="1" pin="GND"/>
+</segment>
 </net>
 <net name="SERIAL_FMU_TO_IO" class="0">
@@
 </segment>
 </net>
-<net name="PRESSURE_SENS" class="0">
-<segment>
-<pinref part="U101" gate="PORTC_L" pin="PC5"/>
-<label x="134.62" y="152.4" size="1.27" layer="95" xref="yes"/>
-<wire x1="134.62" y1="152.4" x2="106.68" y2="152.4" width="0.1524" layer="91"/>
-</segment>
-</net>
 <net name="FMU-UART8_TX" class="0">
 <segment>
@@
 </segment>
 </net>
-<net name="VDD_3V3_SENSORS_EN" class="0">
-<segment>
-<pinref part="U101" gate="PORTE_L" pin="PE3"/>
-<wire x1="175.26" y1="157.48" x2="180.34" y2="157.48" width="0.1524" layer="91"/>
-<label x="180.34" y="157.48" size="1.27" layer="95" xref="yes"/>
-</segment>
-</net>
 <net name="N$23" class="0">
 <segment>
@@
 <segment>
 <pinref part="U101" gate="PORTB_L" pin="PB5"/>
-<wire x1="33.02" y1="96.52" x2="38.1" y2="96.52" width="0.1524" layer="91"/>
-<label x="38.1" y="96.52" size="1.27" layer="95" xref="yes"/>
+<wire x1="33.02" y1="96.52" x2="68.58" y2="96.52" width="0.1524" layer="91"/>
+<pinref part="SJ4" gate="G$1" pin="1"/>
+<wire x1="68.58" y1="86.36" x2="68.58" y2="96.52" width="0.1524" layer="91"/>
 </segment>
 </net>
@@
 <segment>
 <pinref part="U101" gate="PORTB_L" pin="PB7"/>
-<wire x1="33.02" y1="91.44" x2="38.1" y2="91.44" width="0.1524" layer="91"/>
-<label x="38.1" y="91.44" size="1.27" layer="95" xref="yes"/>
+<wire x1="33.02" y1="91.44" x2="58.42" y2="91.44" width="0.1524" layer="91"/>
+<pinref part="SJ4" gate="G$1" pin="3"/>
+<wire x1="58.42" y1="86.36" x2="58.42" y2="91.44" width="0.1524" layer="91"/>
 </segment>
 </net>
@@
 </segment>
 </net>
+<net name="N$14" class="1">
+<segment>
+<pinref part="U101" gate="PORTE_L" pin="PE3"/>
+<wire x1="175.26" y1="157.48" x2="210.82" y2="157.48" width="0.1524" layer="91"/>
+<pinref part="R104" gate="G$1" pin="1"/>
+</segment>
+</net>
+<net name="N$16" class="0">
+<segment>
+<pinref part="U101" gate="PORTC_L" pin="PC5"/>
+<wire x1="106.68" y1="152.4" x2="137.16" y2="152.4" width="0.1524" layer="91"/>
+<pinref part="R103" gate="G$1" pin="1"/>
+</segment>
+</net>
 </nets>
 </sheet>
@@
 Selected R: 220
 Cacluated If @ 5.5V: 10mA</text>
-<text x="127" y="22.86" size="1.778" layer="97">+ SIGNAL
-_</text>
+<text x="124.46" y="25.4" size="1.778" layer="97">Buzzer</text>
 <text x="50.8" y="104.14" size="1.778" layer="91" rot="R90">AMBER</text>
 <text x="63.5" y="104.14" size="1.778" layer="91" rot="R90">GREEN</text>
@@
 <attribute name="BOM" x="215.9" y="119.38" size="1.778" layer="96" rot="R90" display="off"/>
 </instance>
-<instance part="F-BOOT" gate="G$1" x="152.4" y="88.9">
+<instance part="F-BOOT" gate="G$1" x="152.4" y="99.06">
+<attribute name="PARTNO" x="152.4" y="99.06" size="1.778" layer="96" display="off"/>
+<attribute name="BOM" x="152.4" y="99.06" size="1.778" layer="96" display="off"/>
+</instance>
+<instance part="IO-BOOT0" gate="G$1" x="152.4" y="88.9">
 <attribute name="PARTNO" x="152.4" y="88.9" size="1.778" layer="96" display="off"/>
 <attribute name="BOM" x="152.4" y="88.9" size="1.778" layer="96" display="off"/>
 </instance>
-<instance part="IO-BOOT0" gate="G$1" x="152.4" y="78.74">
-<attribute name="PARTNO" x="152.4" y="78.74" size="1.778" layer="96" display="off"/>
-<attribute name="BOM" x="152.4" y="78.74" size="1.778" layer="96" display="off"/>
-</instance>
 <instance part="DP" gate="G$1" x="215.9" y="78.74">
 <attribute name="PARTNO" x="215.9" y="78.74" size="1.778" layer="96" rot="R90" display="off"/>
@@
 <attribute name="BOM" x="215.9" y="109.22" size="1.778" layer="96" rot="R90" display="off"/>
 </instance>
-<instance part="!VBUS_V" gate="G$1" x="152.4" y="119.38">
-<attribute name="PARTNO" x="152.4" y="119.38" size="1.778" layer="96" rot="R90" display="off"/>
-<attribute name="BOM" x="152.4" y="119.38" size="1.778" layer="96" rot="R90" display="off"/>
-</instance>
-<instance part="!VDD_SERVO" gate="G$1" x="152.4" y="109.22">
-<attribute name="PARTNO" x="152.4" y="109.22" size="1.778" layer="96" rot="R90" display="off"/>
-<attribute name="BOM" x="152.4" y="109.22" size="1.778" layer="96" rot="R90" display="off"/>
-</instance>
-<instance part="!VDD_BRICK" gate="G$1" x="152.4" y="99.06">
-<attribute name="PARTNO" x="152.4" y="99.06" size="1.778" layer="96" rot="R90" display="off"/>
-<attribute name="BOM" x="152.4" y="99.06" size="1.778" layer="96" rot="R90" display="off"/>
-</instance>
 <instance part="VDD_5V_IN" gate="G$1" x="215.9" y="99.06">
 <attribute name="PARTNO" x="215.9" y="99.06" size="1.778" layer="96" display="off"/>
@@
 <segment>
 <pinref part="F-BOOT" gate="G$1" pin="P$1"/>
-<wire x1="144.78" y1="88.9" x2="139.7" y2="88.9" width="0.1524" layer="91"/>
-<label x="139.7" y="88.9" size="1.27" layer="95" rot="R180" xref="yes"/>
+<wire x1="144.78" y1="99.06" x2="139.7" y2="99.06" width="0.1524" layer="91"/>
+<label x="139.7" y="99.06" size="1.27" layer="95" rot="R180" xref="yes"/>
 </segment>
 </net>
@@
 <segment>
 <pinref part="IO-BOOT0" gate="G$1" pin="P$1"/>
-<wire x1="144.78" y1="78.74" x2="139.7" y2="78.74" width="0.1524" layer="91"/>
-<label x="139.7" y="78.74" size="1.27" layer="95" rot="R180" xref="yes"/>
+<wire x1="144.78" y1="88.9" x2="139.7" y2="88.9" width="0.1524" layer="91"/>
+<label x="139.7" y="88.9" size="1.27" layer="95" rot="R180" xref="yes"/>
 </segment>
 </net>
@@
 </segment>
 </net>
-<net name="!VBUS_VALID" class="0">
-<segment>
-<pinref part="!VBUS_V" gate="G$1" pin="P$1"/>
-<wire x1="144.78" y1="119.38" x2="139.7" y2="119.38" width="0.1524" layer="91"/>
-<label x="139.7" y="119.38" size="1.27" layer="95" rot="R180" xref="yes"/>
-</segment>
-</net>
-<net name="!VDD_SERVO_VALID" class="0">
-<segment>
-<pinref part="!VDD_SERVO" gate="G$1" pin="P$1"/>
-<wire x1="144.78" y1="109.22" x2="139.7" y2="109.22" width="0.1524" layer="91"/>
-<label x="139.7" y="109.22" size="1.27" layer="95" rot="R180" xref="yes"/>
-</segment>
-</net>
-<net name="!VDD_BRICK_VALID" class="0">
-<segment>
-<pinref part="!VDD_BRICK" gate="G$1" pin="P$1"/>
-<wire x1="144.78" y1="99.06" x2="139.7" y2="99.06" width="0.1524" layer="91"/>
-<label x="139.7" y="99.06" size="1.27" layer="95" rot="R180" xref="yes"/>
-</segment>
-</net>
